Commit message: Adjust position

File: urdf/barista_robot_model.urdf (robot description, URDF)
Before this commit: robot barista_robot, 11 links, 10 joints
Joints:
- joint cup_holder_tray_joint: origin xyz=0 0 0.375 rpy=0 0 0 -> xyz=0 0 0.41 rpy=0 0 0
- joint front_left_rod_joint: origin xyz=0.08 0.08 0.155 rpy=0 0 0 -> xyz=0.08 0.08 0.19 rpy=0 0 0
- joint front_right_rod_joint: origin xyz=0.08 -0.08 0.155 rpy=0 0 0 -> xyz=0.08 -0.08 0.19 rpy=0 0 0
- joint laser_joint: origin xyz=0.13 0 0.155 rpy=0 0 0 -> xyz=0.13 0 0.19 rpy=0 0 0
- joint left_wheel_joint: origin xyz=0 0.178 0.0352 rpy=0 0 0 -> xyz=0 0.14 0.0352 rpy=0 0 0
- joint rear_left_rod_joint: origin xyz=-0.08 0.08 0.155 rpy=0 0 0 -> xyz=-0.08 0.08 0.19 rpy=0 0 0
- joint rear_right_rod_joint: origin xyz=-0.08 -0.08 0.155 rpy=0 0 0 -> xyz=-0.08 -0.08 0.19 rpy=0 0 0
- joint right_wheel_joint: origin xyz=0 -0.178 0.0352 rpy=0 0 0 -> xyz=0 -0.14 0.0352 rpy=0 0 0

Commit message: Adjust position

File: urdf/barista_robot_model.urdf (robot description, URDF)
Before this commit: robot barista_robot, 11 links, 10 joints
Joints:
- joint cup_holder_tray_joint: origin xyz=0 0 0.41 rpy=0 0 0 -> xyz=0 0 0.2975 rpy=0 0 0
- joint front_caster_joint: origin xyz=0.12 0 0.025 rpy=0 0 0 -> xyz=0.12 0 -0.0875 rpy=0 0 0
- joint front_left_rod_joint: origin xyz=0.08 0.08 0.19 rpy=0 0 0 -> xyz=0.08 0.08 0.0775 rpy=0 0 0
- joint front_right_rod_joint: origin xyz=0.08 -0.08 0.19 rpy=0 0 0 -> xyz=0.08 -0.08 0.0775 rpy=0 0 0
- joint laser_joint: origin xyz=0.13 0 0.19 rpy=0 0 0 -> xyz=0.13 0 0.0775 rpy=0 0 0
- joint left_wheel_joint: origin xyz=0 0.14 0.0352 rpy=0 0 0 -> xyz=0 0.14 -0.0775 rpy=0 0 0
- joint rear_caster_joint: origin xyz=-0.12 0 0.025 rpy=0 0 0 -> xyz=-0.12 0 -0.0875 rpy=0 0 0
- joint rear_left_rod_joint: origin xyz=-0.08 0.08 0.19 rpy=0 0 0 -> xyz=-0.08 0.08 0.0775 rpy=0 0 0
- joint rear_right_rod_joint: origin xyz=-0.08 -0.08 0.19 rpy=0 0 0 -> xyz=-0.08 -0.08 0.0775 rpy=0 0 0
- joint right_wheel_joint: origin xyz=0 -0.14 0.0352 rpy=0 0 0 -> xyz=0 -0.14 -0.0775 rpy=0 0 0

Commit message: Add mesh scale

File: urdf/barista_robot_model.urdf (robot description, URDF)
Before this commit: robot barista_robot, 11 links, 10 joints
Links:
- link laser_link: geometry collision box size=0.05 0.05 0.05; visual mesh filename=package://barista_robot_description/meshes/hokuyo.dae scale=1 1 1

Commit message: Modify rods position

File: urdf/barista_robot_model.urdf (robot description, URDF)
Before this commit: robot barista_robot, 11 links, 10 joints
Joints:
- joint front_left_rod_joint: origin xyz=0.08 0.08 0.0775 rpy=0 0 0 -> xyz=0.03 0.13 0.0775 rpy=0 0 0
- joint front_right_rod_joint: origin xyz=0.08 -0.08 0.0775 rpy=0 0 0 -> xyz=0.03 -0.13 0.0775 rpy=0 0 0
- joint rear_left_rod_joint: origin xyz=-0.08 0.08 0.0775 rpy=0 0 0 -> xyz=-0.03 0.13 0.0775 rpy=0 0 0
- joint rear_right_rod_joint: origin xyz=-0.08 -0.08 0.0775 rpy=0 0 0 -> xyz=-0.03 -0.13 0.0775 rpy=0 0 0

Commit message: Adjust laser scanner ray height

File: urdf/barista_robot_model.urdf (robot description, URDF)
Before this commit: robot barista_robot, 11 links, 10 joints
Joints:
- joint laser_joint: origin xyz=0.13 0 0.0775 rpy=0 0 0 -> xyz=0.13 0 0.11 rpy=0 0 0
