Commit message: Adjust position

File: xacro/barista_robot_model.urdf.xacro (robot description, xacro)
@@ -25,10 +25,10 @@
   <link name="base_link">
     <inertial>
-      <origin xyz="0 0 0.1125" rpy="0 0 0"/>
+      <origin xyz="0 0 0" rpy="0 0 0"/>
       <mass value="5.0"/>
       <inertia ixx="0.1" ixy="0" ixz="0" iyy="0.1" iyz="0" izz="0.1"/>
     </inertial>
     <visual>
-      <origin xyz="0 0 0.1125" rpy="0 0 0"/>
+      <origin xyz="0 0 0" rpy="0 0 0"/>
       <geometry>
         <cylinder radius="0.178" length="0.155"/>
@@ -37,5 +37,5 @@
     </visual>
     <collision>
-      <origin xyz="0 0 0.1125" rpy="0 0 0"/>
+      <origin xyz="0 0 0" rpy="0 0 0"/>
       <geometry>
         <cylinder radius="0.178" length="0.155"/>

File: xacro/caster_wheel.xacro (robot description, xacro)
@@ -35,5 +35,5 @@
       <parent link="base_link"/>
       <child link="${prefix}_caster_link"/>
-      <origin xyz="${x_offset} ${y_offset} ${caster_radius}" rpy="0 0 0"/>
+      <origin xyz="${x_offset} ${y_offset} -0.0875" rpy="0 0 0"/>
     </joint>
     <!-- Gazebo-specific properties -->

File: xacro/cup_holder_tray.xacro (robot description, xacro)
@@ -7,5 +7,4 @@
     <xacro:property name="tray_height" value="0.09" />
     <xacro:property name="tray_mass" value="1.0" />
-    <xacro:property name="tray_z_offset" value="0.41" />
     <link name="cup_holder_tray_link">
       <inertial>
@@ -37,5 +36,5 @@
       <parent link="base_link"/>
       <child link="cup_holder_tray_link"/>
-      <origin xyz="0 0 ${tray_z_offset}" rpy="0 0 0"/>
+      <origin xyz="0 0 0.2975" rpy="0 0 0"/>
     </joint>
     <!-- Gazebo-specific properties -->

File: xacro/drive_wheel.xacro (robot description, xacro)
@@ -37,5 +37,5 @@
       <parent link="base_link"/>
       <child link="${prefix}_wheel_link"/>
-      <origin xyz="0 ${reflect * wheel_joint_offset_y} ${wheel_radius}" rpy="0 0 0"/>
+      <origin xyz="0 ${reflect * wheel_joint_offset_y} -0.0775" rpy="0 0 0"/>
       <axis xyz="0 1 0"/>
     </joint>

File: xacro/laser_scanner.xacro (robot description, xacro)
@@ -7,5 +7,4 @@
     <xacro:property name="laser_x_offset" value="0.13" />
     <xacro:property name="laser_y_offset" value="0.0" />
-    <xacro:property name="laser_z_offset" value="0.19" />
     <link name="laser_link">
       <inertial>
@@ -31,5 +30,5 @@
       <parent link="base_link"/>
       <child link="laser_link"/>
-      <origin xyz="${laser_x_offset} ${laser_y_offset} ${laser_z_offset}" rpy="0 0 0"/>
+      <origin xyz="${laser_x_offset} ${laser_y_offset} 0.0775" rpy="0 0 0"/>
     </joint>
     <!-- Gazebo-specific properties -->

File: xacro/standoff_rod.xacro (robot description, xacro)
@@ -37,5 +37,5 @@
       <parent link="base_link"/>
       <child link="${prefix}_rod_link"/>
-      <origin xyz="${x_offset} ${y_offset} ${rod_z_offset}" rpy="0 0 0"/>
+      <origin xyz="${x_offset} ${y_offset} 0.0775" rpy="0 0 0"/>
     </joint>
     <!-- Gazebo-specific properties -->

Commit message: Modify robot color property

File: xacro/barista_robot_model.urdf.xacro (robot description, xacro)
@@ -7,9 +7,20 @@
   <xacro:include filename="$(find barista_robot_description)/xacro/cup_holder_tray.xacro" />
   <xacro:include filename="$(find barista_robot_description)/xacro/laser_scanner.xacro" />
-  <!-- Define argument for laser scanner inclusion -->
+  <!-- Define arguments -->
   <xacro:arg name="include_laser" default="true"/>
+  <xacro:arg name="robot_color" default="Blue"/>
+  <!-- Set color property based on the robot_color parameter -->
+  <xacro:property name="robot_gazebo_color" value="Blue"/>
+  <xacro:property name="robot_visual_color" value="robot_blue"/>
+  <xacro:if value="${'$(arg robot_color)' == 'Red'}">
+    <xacro:property name="robot_gazebo_color" value="Red"/>
+    <xacro:property name="robot_visual_color" value="robot_red"/>
+  </xacro:if>
   <!-- Define colors -->
   <material name="robot_blue">
     <color rgba="0.0 0.0 0.8 1.0"/>
+  </material>
+  <material name="robot_red">
+    <color rgba="0.8 0.0 0.0 1.0"/>
   </material>
   <material name="robot_black">
@@ -34,5 +45,5 @@
         <cylinder radius="0.178" length="0.155"/>
       </geometry>
-      <material name="robot_blue"/>
+      <material name="${robot_visual_color}"/>
     </visual>
     <collision>
@@ -45,5 +56,5 @@
   <!-- Gazebo color for the base_link -->
   <gazebo reference="base_link">
-    <material>Gazebo/Blue</material>
+    <material>Gazebo/${robot_gazebo_color}</material>
   </gazebo>
   <!-- Add wheels using macros -->
@@ -59,5 +70,5 @@
   <xacro:standoff_rod prefix="rear_right" x_offset="-0.03" y_offset="-0.13" />
   <!-- Add cup holder tray using macro -->
-  <xacro:cup_holder_tray />
+  <xacro:cup_holder_tray robot_color="$(arg robot_color)" />
   <!-- Add laser scanner if include_laser is true -->
   <xacro:if value="$(arg include_laser)">
@@ -68,4 +79,5 @@
     <plugin name="gazebo_ros_diff_drive" filename="libgazebo_ros_diff_drive.so">
       <ros>
+        <!-- Namespace will be automatically prefixed by the robot's namespace -->
         <namespace>/</namespace>
       </ros>

Commit message: Edit namespace

File: xacro/barista_robot_model.urdf.xacro (robot description, xacro)
@@ -10,4 +10,7 @@
   <xacro:arg name="include_laser" default="true"/>
   <xacro:arg name="robot_color" default="Blue"/>
+  <xacro:arg name="robot_name" default="barista"/>
+  <!-- Set robot_name property based on the argument -->
+  <xacro:property name="robot_name" value="$(arg robot_name)"/>
   <!-- Set color property based on the robot_color parameter -->
   <xacro:property name="robot_gazebo_color" value="Blue"/>
@@ -80,5 +83,7 @@
       <ros>
         <!-- Namespace will be automatically prefixed by the robot's namespace -->
-        <namespace>/</namespace>
+        <namespace>/${robot_name}</namespace>
+        <remapping>cmd_vel:=cmd_vel</remapping>
+        <remapping>odom:=odom</remapping>
       </ros>
       <update_rate>100.0</update_rate>
@@ -94,6 +99,6 @@
       <publish_wheel_tf>false</publish_wheel_tf>
       <odometry_topic>odom</odometry_topic>
-      <odometry_frame>odom</odometry_frame>
-      <robot_base_frame>base_link</robot_base_frame>
+      <odometry_frame>${robot_name}/odom</odometry_frame>
+      <robot_base_frame>${robot_name}/base_link</robot_base_frame>
     </plugin>
   </gazebo>
