Commit message: Add mesh scale

File: xacro/laser_scanner.xacro (robot description, xacro)
@@ -16,5 +16,5 @@
         <origin xyz="0 0 0.025" rpy="0 0 0"/>
         <geometry>
-          <mesh filename="package://barista_robot_description/meshes/hokuyo.dae"/>
+          <mesh filename="package://barista_robot_description/meshes/hokuyo.dae" scale="1 1 1"/>
         </geometry>
         <material name="robot_black"/>
@@ -34,5 +34,5 @@
     <!-- Gazebo-specific properties -->
     <gazebo reference="laser_link">
-      <material>Gazebo/Black</material>
+      <material>Gazebo/Grey</material>
       <sensor type="ray" name="head_hokuyo_sensor">
         <pose>0 0 0 0 0 0</pose>

Commit message: Adjust laser scanner ray height

File: xacro/laser_scanner.xacro (robot description, xacro)
@@ -9,17 +9,17 @@
     <link name="laser_link">
       <inertial>
-        <origin xyz="0 0 0.025" rpy="0 0 0"/>
+        <origin xyz="0 0 0" rpy="0 0 0"/>
         <mass value="${laser_mass}"/>
         <inertia ixx="0.0001" ixy="0" ixz="0" iyy="0.0001" iyz="0" izz="0.0001"/>
       </inertial>
       <visual>
-        <origin xyz="0 0 0.025" rpy="0 0 0"/>
+        <origin xyz="0 0 0" rpy="0 0 0"/>
         <geometry>
-          <mesh filename="package://barista_robot_description/meshes/hokuyo.dae" scale="1 1 1"/>
+          <mesh filename="package://barista_robot_description/meshes/hokuyo.dae"/>
         </geometry>
         <material name="robot_black"/>
       </visual>
       <collision>
-        <origin xyz="0 0 0.025" rpy="0 0 0"/>
+        <origin xyz="0 0 0" rpy="0 0 0"/>
         <geometry>
           <box size="0.05 0.05 0.05"/>
@@ -30,5 +30,5 @@
       <parent link="base_link"/>
       <child link="laser_link"/>
-      <origin xyz="${laser_x_offset} ${laser_y_offset} 0.0775" rpy="0 0 0"/>
+      <origin xyz="${laser_x_offset} ${laser_y_offset} 0.11" rpy="0 0 0"/>
     </joint>
     <!-- Gazebo-specific properties -->
@@ -39,4 +39,5 @@
         <visualize>true</visualize>
         <update_rate>20</update_rate>
+        <always_on>true</always_on>
         <ray>
           <scan>
@@ -66,5 +67,4 @@
           <output_type>sensor_msgs/LaserScan</output_type>
           <frame_name>laser_link</frame_name>
-          <visualize>true</visualize>
         </plugin>
       </sensor>

Commit message: Edit namespace

File: xacro/laser_scanner.xacro (robot description, xacro)
@@ -7,4 +7,7 @@
     <xacro:property name="laser_x_offset" value="0.13" />
     <xacro:property name="laser_y_offset" value="0.0" />
+    <xacro:arg name="robot_name" default="barista"/>
+    <!-- Set robot_name property based on the argument -->
+    <xacro:property name="robot_name" value="$(arg robot_name)"/>
     <link name="laser_link">
       <inertial>
@@ -61,9 +64,9 @@
         <plugin name="gazebo_ros_head_hokuyo_controller" filename="libgazebo_ros_ray_sensor.so">
           <ros>
-            <namespace>/</namespace>
+            <namespace>/${robot_name}</namespace>
             <remapping>~/out:=scan</remapping>
           </ros>
           <output_type>sensor_msgs/LaserScan</output_type>
-          <frame_name>laser_link</frame_name>
+          <frame_name>${robot_name}/laser_link</frame_name>
         </plugin>
       </sensor>
